File: hardware/breakout.kicad_pcb (KiCad board)
At the start: 2 copper layers, 40.3 x 50 mm, 7 parts, among them J1 Conn_01x18_Male, J2 Conn_Coaxial, J3 Conn_01x18_Male, J4 Conn_Coaxial, U1 RFM95W-915S2

Commit message: [add] Push button for manual rseet
Parts:
- added SW1: SW_Push, KiCad/kicad-footprints/Button_Switch_SMD.pretty:SW_DIP_SPSTx01_Slide_6.7x4.1mm_W8.61mm_P2.54mm_LowProfile, F.Cu at (145.8, 93.5)
- C1: moved to F.Cu
- moved C1 17.6 mm to (136.0, 120.4), turned to 90 degrees
Routing:
- net GND: track 88.2 -> 50.9 mm, vias 2 -> 0
- net Net-(J1-Pad9): track 31.4 -> 22.2 mm
- net +3V3: track 35.9 -> 31.0 mm
- net /RST: track 46.6 -> 46.5 mm, vias 0 -> 1
- added copper zone on F.Cu, net GND
